Commit message: scripts in the src folder

File: description/gazebo_ros2_control_plugin.xacro (robot description, xacro)
@@ -1,4 +1,5 @@
 <?xml version="1.0"?>
 <robot xmlns:xacro="http://www.ros.org/wiki/xacro">
+    <xacro:arg name="imu_visual"    default="false"/>
 <!-- ************* JOINT CONTROLLER GAZEBO PLUGIN ************** -->
     <!--

File: description/hyperdog_gazebo.xacro (robot description, xacro)
@@ -11,4 +11,39 @@
 -->
     <xacro:include filename="physics.xacro" />
+    <gazebo reference="imu_link">
+        <sensor type="imu" name="imu">
+          <always_on>true</always_on>
+          <visualize>$(arg imu_visual)</visualize>
+        </sensor>
+        <material>Gazebo/Grey</material>
+    </gazebo>
+    <gazebo>
+        <plugin name="imu_plugin" filename="libgazebo_ros_imu.so">
+          <alwaysOn>true</alwaysOn>
+          <bodyName>imu_link</bodyName>
+          <frameName>imu_link</frameName>
+          <topicName>imu</topicName>
+          <serviceName>imu_service</serviceName>
+          <gaussianNoise>0.0</gaussianNoise>
+          <updateRate>0</updateRate>
+          <imu>
+            <noise>
+              <type>gaussian</type>
+              <rate>
+                <mean>0.0</mean>
+                <stddev>2e-4</stddev>
+                <bias_mean>0.0000075</bias_mean>
+                <bias_stddev>0.0000008</bias_stddev>
+              </rate>
+              <accel>
+                <mean>0.0</mean>
+                <stddev>1.7e-2</stddev>
+                <bias_mean>0.1</bias_mean>
+                <bias_stddev>0.001</bias_stddev>
+              </accel>
+            </noise>
+          </imu>
+        </plugin>
+      </gazebo>
     <xacro:macro name="gz_hip">
         <mu1>0.2</mu1>

File: description/hyperdog_urdf_links.xacro (robot description, xacro)
@@ -52,4 +52,10 @@
         </collision>
     </link>
+    <joint name="imu_joint" type="fixed">
+        <parent link="base_link"/>
+        <child link="imu_link"/>
+        <origin xyz="0.0 0 0.068" rpy="0 0 0"/>
+      </joint>
+      <link name="imu_link"/>
     <!-- !!!!!!!!!!!!!!!!!!!!!!! HIPS !!!!!!!!!!!!!!!!!!!!!!!!!!!! -->
     <!-- *********** FR_hip *********** -->
