Commit message: script changes

File: description/depthcam.xacro (robot description, xacro)
@@ -1,32 +1,26 @@
 <?xml version="1.0"?>
 <robot xmlns:xacro="http://www.ros.org/wiki/xacro" >
-    <joint name="camera_joint" type="fixed">
+    <joint name="camera_joint_depth" type="fixed">
         <parent link="base_link"/>
-        <child link="camera_link"/>
+        <child link="camera_link_depth"/>
         <origin xyz="0.12 0 0.10" rpy="0 0 0"/>
     </joint>
-    <link name="camera_link">
+    <link name="camera_link_depth">
         <visual>
             <geometry>
                 <box size="0.010 0.03 0.03"/>
             </geometry>
-            <material name="black"/>
-        </visual>
-        <visual>
-            <origin xyz="0 0 -0.05"/>
-            <geometry>
-                <cylinder radius="0.002" length="0.1"/>
-            </geometry>
+            <material name="red"/>
         </visual>
     </link>
-    <joint name="camera_optical_joint" type="fixed">
-        <parent link="camera_link"/>
-        <child link="camera_link_optical"/>
+    <joint name="camera_optical_joint_depth" type="fixed">
+        <parent link="camera_link_depth"/>
+        <child link="camera_link_optical_depth"/>
         <origin xyz="0 0 0" rpy="${-pi/2} 0 ${-pi/2}"/>
     </joint>
-    <link name="camera_link_optical"></link>
-    <!-- <gazebo reference="camera_link">
-        <material>Gazebo/Black</material>
-        <sensor name="camera" type="camera">
+    <link name="camera_link_optical_depth"></link>
+    <gazebo reference="camera_link_depth">
+        <material>Gazebo/Red</material>
+        <sensor name="camera" type="depth">
             <pose> 0 0 0 0 0 0 </pose>
             <visualize>true</visualize>
@@ -35,5 +29,5 @@
                 <horizontal_fov>1.089</horizontal_fov>
                 <image>
-                    <format>R8G8B8</format>
+                    <format>B8G8R8</format>
                     <width>640</width>
                     <height>480</height>
@@ -45,7 +39,9 @@
             </camera>
             <plugin name="camera_controller" filename="libgazebo_ros_camera.so">
-                <frame_name>camera_link_optical</frame_name>
+                <frame_name>camera_link_optical_depth</frame_name>
+                <min_depth>0.1</min_depth>
+                <max_depth>100.0</max_depth>
             </plugin>
         </sensor>
-    </gazebo> -->
+    </gazebo>
 </robot>

File: description/hyperdog.urdf.xacro (robot description, xacro)
@@ -10,3 +10,4 @@
     <xacro:include filename="gazebo_ros2_control_plugin.xacro" />
     <xacro:include filename="camera.xacro" />
+    <xacro:include filename="depthcam.xacro"/>
 </robot>

File: description/hyperdog_gazebo.xacro (robot description, xacro)
@@ -2,4 +2,5 @@
 <robot xmlns:xacro="http://www.ros.org/wiki/xacro">
     <xacro:arg name="imu_visual"    default="false"/>
+    <xacro:arg name="camera_visual" default="false"/>
 <!--
     _____________________________________________________________________

File: description/hyperdog_urdf_links.xacro (robot description, xacro)
@@ -1,4 +1,8 @@
 <?xml version="1.0"?>
 <robot xmlns:xacro="http://www.ros.org/wiki/xacro">
+    <xacro:property name="r200_cam_rgb_px" value="0.005"/>
+    <xacro:property name="r200_cam_rgb_py" value="0.018"/>
+    <xacro:property name="r200_cam_rgb_pz" value="0.013"/>
+    <xacro:property name="r200_cam_depth_offset" value="0.01"/>
 <!--
     * Autor: nipun.dhananjaya@gmail.com
