Commit message: new version

File: description/consts.xacro (robot description, xacro)
@@ -8,36 +8,36 @@
     <xacro:property name="lleg_low_limit" value="-1.57"/>
     <xacro:property name="lleg_up_limit"  value="2.618"/>
-    <xacro:property name="velocity"       value="1"/>
-    <xacro:property name="effort"         value="10"/>
+    <xacro:property name="velocity"       value="3"/>
+    <xacro:property name="effort"         value="3"/>
     <!-- joint dynamics -->
     <xacro:property name="use_dynamics" value="true"/>
     <xacro:macro name="hip_joint_dynamics">
-        <dynamics damping="0.01" friction="10000"/>
+        <dynamics damping="0.1" friction="10000"/>
     </xacro:macro>
     <xacro:macro name="uleg_joint_dynamics">
-        <dynamics damping="0.01" friction="10000"/>
+        <dynamics damping="0.1" friction="10000"/>
     </xacro:macro>
     <xacro:macro name="lleg_joint_dynamics">
-        <dynamics damping="0.01" friction="10000"/>
+        <dynamics damping="0.1" friction="10000"/>
     </xacro:macro>
     <!-- configure inertia -->
-    <xacro:property name="body_mass" value="3"/>
+    <xacro:property name="body_mass" value="14"/>
     <xacro:property name="body_inertia_x_len" value="0.28"/>
     <xacro:property name="body_inertia_y_len" value="0.172"/>
     <xacro:property name="body_inertia_z_len" value="0.04"/>
-    <xacro:property name="hip_mass" value="0.3"/>
+    <xacro:property name="hip_mass" value="1"/>
     <xacro:property name="hip_inertia_x_len" value="0.05"/>
     <xacro:property name="hip_inertia_y_len" value="0.03"/>
     <xacro:property name="hip_inertia_z_len" value="0.04"/>
-    <xacro:property name="uleg_mass" value="0.5"/>
+    <xacro:property name="uleg_mass" value="1"/>
     <xacro:property name="uleg_inertia_x_len" value="0.14"/>
     <xacro:property name="uleg_inertia_y_len" value="0.01"/>
     <xacro:property name="uleg_inertia_z_len" value="0.01"/>
-    <xacro:property name="lleg_mass" value="0.2"/>
+    <xacro:property name="lleg_mass" value="1"/>
     <xacro:property name="lleg_inertia_x_len" value="0.08"/>
     <xacro:property name="lleg_inertia_y_len" value="0.001"/>
     <xacro:property name="lleg_inertia_z_len" value="0.005"/>
     <!-- feet -->
-    <xacro:property name="foot_mass" value="0.1"/>
+    <xacro:property name="foot_mass" value="0.5"/>
     <xacro:property name="foot_radius" value="0.02"/>
 </robot>

File: description/gazebo_ros2_control_plugin.xacro (robot description, xacro)
@@ -7,4 +7,5 @@
         </hardware>
         <joint name="FR_hip_joint">
+            <limit  velocity="3" effort="3"/> <!-- effort = 7 -->
             <command_interface name="position">
                 <param name="min">-1.57</param>
@@ -18,4 +19,5 @@
         </joint>
         <joint name="FR_uleg_joint">
+            <limit  velocity="3" effort="3"/>
             <command_interface name="position">
                 <param name="min">-1.2217</param>
@@ -29,4 +31,5 @@
         </joint>
         <joint name="FR_lleg_joint">
+            <limit  velocity="3" effort="3"/>
             <command_interface name="position">
                 <param name="min">0.45</param>
@@ -40,4 +43,5 @@
         </joint>
         <joint name="FL_hip_joint">
+            <limit  velocity="3" effort="3"/>
             <command_interface name="position">
                 <param name="min">-1.57</param>
@@ -51,4 +55,5 @@
         </joint>
         <joint name="FL_uleg_joint">
+            <limit  velocity="3" effort="3"/>
             <command_interface name="position">
                 <param name="min">-1.2217</param>
@@ -62,4 +67,5 @@
         </joint>
         <joint name="FL_lleg_joint">
+            <limit  velocity="3" effort="3"/>
             <command_interface name="position">
                 <param name="min">0.45</param>
@@ -73,4 +79,5 @@
         </joint>
         <joint name="BR_hip_joint">
+            <limit  velocity="3" effort="3"/>
             <command_interface name="position">
                 <param name="min">-1.57</param>
@@ -84,4 +91,5 @@
         </joint>
         <joint name="BR_uleg_joint">
+            <limit  velocity="3" effort="3"/>
             <command_interface name="position">
                 <param name="min">-1.2217</param>
@@ -95,4 +103,5 @@
         </joint>
         <joint name="BR_lleg_joint">
+            <limit  velocity="3" effort="3"/>
             <command_interface name="position">
                 <param name="min">0.45</param>
@@ -106,4 +115,5 @@
         </joint>
         <joint name="BL_hip_joint">
+            <limit  velocity="3" effort="3"/>
             <command_interface name="position">
                 <param name="min">-1.57</param>
@@ -117,4 +127,5 @@
         </joint>
         <joint name="BL_uleg_joint">
+            <limit  velocity="3" effort="3"/>
             <command_interface name="position">
                 <param name="min">-1.2217</param>
@@ -128,4 +139,5 @@
         </joint>
         <joint name="BL_lleg_joint">
+            <limit  velocity="3" effort="3"/>
             <command_interface name="position">
                 <param name="min">0.45</param>

File: description/hyperdog.urdf.xacro (robot description, xacro)
@@ -9,5 +9,4 @@
     <xacro:include filename="hyperdog_gazebo.xacro" />
     <xacro:include filename="gazebo_ros2_control_plugin.xacro" />
-    <xacro:include filename="camera.xacro" />
-    <xacro:include filename="depthcam.xacro"/>
+    <xacro:include filename="lidar.xacro"/>
 </robot>
