Commit message: new version

File: description/consts.xacro (robot description, xacro)
@@ -8,36 +8,36 @@
     <xacro:property name="lleg_low_limit" value="-1.57"/>
     <xacro:property name="lleg_up_limit"  value="2.618"/>
-    <xacro:property name="velocity"       value="3"/>
+    <xacro:property name="velocity"       value="1"/>
     <xacro:property name="effort"         value="3"/>
     <!-- joint dynamics -->
     <xacro:property name="use_dynamics" value="true"/>
     <xacro:macro name="hip_joint_dynamics">
-        <dynamics damping="0.1" friction="10000"/>
+        <dynamics damping="0.01" friction="10000"/>
     </xacro:macro>
     <xacro:macro name="uleg_joint_dynamics">
-        <dynamics damping="0.1" friction="10000"/>
+        <dynamics damping="0.01" friction="10000"/>
     </xacro:macro>
     <xacro:macro name="lleg_joint_dynamics">
-        <dynamics damping="0.1" friction="10000"/>
+        <dynamics damping="0.01" friction="10000"/>
     </xacro:macro>
     <!-- configure inertia -->
-    <xacro:property name="body_mass" value="14"/>
+    <xacro:property name="body_mass" value="3"/>
     <xacro:property name="body_inertia_x_len" value="0.28"/>
     <xacro:property name="body_inertia_y_len" value="0.172"/>
     <xacro:property name="body_inertia_z_len" value="0.04"/>
-    <xacro:property name="hip_mass" value="1"/>
+    <xacro:property name="hip_mass" value="0.3"/>
     <xacro:property name="hip_inertia_x_len" value="0.05"/>
     <xacro:property name="hip_inertia_y_len" value="0.03"/>
     <xacro:property name="hip_inertia_z_len" value="0.04"/>
-    <xacro:property name="uleg_mass" value="1"/>
+    <xacro:property name="uleg_mass" value="0.5"/>
     <xacro:property name="uleg_inertia_x_len" value="0.14"/>
     <xacro:property name="uleg_inertia_y_len" value="0.01"/>
     <xacro:property name="uleg_inertia_z_len" value="0.01"/>
-    <xacro:property name="lleg_mass" value="1"/>
+    <xacro:property name="lleg_mass" value="0.2"/>
     <xacro:property name="lleg_inertia_x_len" value="0.08"/>
     <xacro:property name="lleg_inertia_y_len" value="0.001"/>
     <xacro:property name="lleg_inertia_z_len" value="0.005"/>
     <!-- feet -->
-    <xacro:property name="foot_mass" value="0.5"/>
+    <xacro:property name="foot_mass" value="0.1"/>
     <xacro:property name="foot_radius" value="0.02"/>
 </robot>

File: description/gazebo_ros2_control_plugin.xacro (robot description, xacro)
@@ -1,4 +1,11 @@
 <?xml version="1.0"?>
 <robot xmlns:xacro="http://www.ros.org/wiki/xacro">
+<!-- ************* JOINT CONTROLLER GAZEBO PLUGIN ************** -->
+    <!--
+    _____________________________________________________________________
+        include this file into: /description/hyperdog.urdf.xacro
+        using following line:
+                    <xacro:include filename="gazebo_ros2_control_plugin.xacro" />
+    _____________________________________________________________________ -->
     <!-- CONFIGURE JOINTS OF THE ROBOT -->
     <ros2_control name="GazeboSystem" type="System">
@@ -7,5 +14,4 @@
         </hardware>
         <joint name="FR_hip_joint">
-            <limit  velocity="3" effort="3"/> <!-- effort = 7 -->
             <command_interface name="position">
                 <param name="min">-1.57</param>
@@ -19,5 +25,4 @@
         </joint>
         <joint name="FR_uleg_joint">
-            <limit  velocity="3" effort="3"/>
             <command_interface name="position">
                 <param name="min">-1.2217</param>
@@ -31,5 +36,4 @@
         </joint>
         <joint name="FR_lleg_joint">
-            <limit  velocity="3" effort="3"/>
             <command_interface name="position">
                 <param name="min">0.45</param>
@@ -43,5 +47,4 @@
         </joint>
         <joint name="FL_hip_joint">
-            <limit  velocity="3" effort="3"/>
             <command_interface name="position">
                 <param name="min">-1.57</param>
@@ -55,5 +58,4 @@
         </joint>
         <joint name="FL_uleg_joint">
-            <limit  velocity="3" effort="3"/>
             <command_interface name="position">
                 <param name="min">-1.2217</param>
@@ -67,5 +69,4 @@
         </joint>
         <joint name="FL_lleg_joint">
-            <limit  velocity="3" effort="3"/>
             <command_interface name="position">
                 <param name="min">0.45</param>
@@ -79,5 +80,4 @@
         </joint>
         <joint name="BR_hip_joint">
-            <limit  velocity="3" effort="3"/>
             <command_interface name="position">
                 <param name="min">-1.57</param>
@@ -91,5 +91,4 @@
         </joint>
         <joint name="BR_uleg_joint">
-            <limit  velocity="3" effort="3"/>
             <command_interface name="position">
                 <param name="min">-1.2217</param>
@@ -103,5 +102,4 @@
         </joint>
         <joint name="BR_lleg_joint">
-            <limit  velocity="3" effort="3"/>
             <command_interface name="position">
                 <param name="min">0.45</param>
@@ -115,5 +113,4 @@
         </joint>
         <joint name="BL_hip_joint">
-            <limit  velocity="3" effort="3"/>
             <command_interface name="position">
                 <param name="min">-1.57</param>
@@ -127,5 +124,4 @@
         </joint>
         <joint name="BL_uleg_joint">
-            <limit  velocity="3" effort="3"/>
             <command_interface name="position">
                 <param name="min">-1.2217</param>
@@ -139,5 +135,4 @@
         </joint>
         <joint name="BL_lleg_joint">
-            <limit  velocity="3" effort="3"/>
             <command_interface name="position">
                 <param name="min">0.45</param>

File: description/hyperdog.urdf.xacro (robot description, xacro)
@@ -6,7 +6,6 @@
     <xacro:include filename="hyperdog_urdf_joints.xacro" />
     <!-- ****************   INCLUDES OTHER FILES  ******************* -->
-    <!-- <xacro:include filename="gazebo_ros2_control_plugin.xacro" />  -->
+    <xacro:include filename="gazebo_ros2_control_plugin.xacro" />
     <xacro:include filename="hyperdog_gazebo.xacro" />
-    <xacro:include filename="gazebo_ros2_control_plugin.xacro" />
     <xacro:include filename="lidar.xacro"/>
 </robot>

File: description/hyperdog_gazebo.xacro (robot description, xacro)
@@ -2,5 +2,4 @@
 <robot xmlns:xacro="http://www.ros.org/wiki/xacro">
     <xacro:arg name="imu_visual"    default="false"/>
-    <xacro:arg name="camera_visual" default="false"/>
 <!--
     _____________________________________________________________________

File: description/hyperdog_urdf_links.xacro (robot description, xacro)
@@ -1,8 +1,4 @@
 <?xml version="1.0"?>
 <robot xmlns:xacro="http://www.ros.org/wiki/xacro">
-    <xacro:property name="r200_cam_rgb_px" value="0.005"/>
-    <xacro:property name="r200_cam_rgb_py" value="0.018"/>
-    <xacro:property name="r200_cam_rgb_pz" value="0.013"/>
-    <xacro:property name="r200_cam_depth_offset" value="0.01"/>
 <!--
     * Autor: nipun.dhananjaya@gmail.com
@@ -61,5 +57,5 @@
         <origin xyz="0.0 0 0.068" rpy="0 0 0"/>
       </joint>
-      <link name="imu_link"/>
+    <link name="imu_link"/>
     <!-- !!!!!!!!!!!!!!!!!!!!!!! HIPS !!!!!!!!!!!!!!!!!!!!!!!!!!!! -->
     <!-- *********** FR_hip *********** -->
@@ -75,4 +71,13 @@
         </visual>
         <collision>
+            <surface>
+                <friction>
+                    <ode>
+                        <mu>0.7</mu>
+                        <mu2>0.7</mu2>
+                        <fdir1>1 0 0</fdir1>
+                    </ode>
+                </friction>
+            </surface>
             <origin xyz="0 0 0" rpy="0 0 0"/>
             <geometry>
@@ -94,4 +99,13 @@
         </visual>
         <collision>
+            <surface>
+                <friction>
+                    <ode>
+                        <mu>0.7</mu>
+                        <mu2>0.7</mu2>
+                        <fdir1>1 0 0</fdir1>
+                    </ode>
+                </friction>
+            </surface>
             <origin xyz="0 0 0" rpy="0 0 0"/>
             <geometry>
@@ -114,5 +128,23 @@
         <collision>
             <origin xyz="0 0 0" rpy="0 0 0"/>
-            <geometry>
+            <surface>
+                <friction>
+                    <ode>
+                        <mu>0.7</mu>
+                        <mu2>0.7</mu2>
+                        <fdir1>1 0 0</fdir1>
+                    </ode>
+                </friction>
+            </surface>
+            <geometry>
+                 <surface>
+                <friction>
+                    <ode>
+                        <mu>0.7</mu>
+                        <mu2>0.7</mu2>
+                        <fdir1>1 0 0</fdir1>
+                    </ode>
+                </friction>
+            </surface>
                 <xacro:rightHip_mesh></xacro:rightHip_mesh>
             </geometry>
@@ -132,4 +164,13 @@
         </visual>
         <collision>
+            <surface>
+                <friction>
+                    <ode>
+                        <mu>0.7</mu>
+                        <mu2>0.7</mu2>
+                        <fdir1>1 0 0</fdir1>
+                    </ode>
+                </friction>
+            </surface>
             <origin xyz="0 0 0" rpy="0 0 0"/>
             <geometry>
@@ -152,4 +193,13 @@
         </visual>
         <collision>
+            <surface>
+                <friction>
+                    <ode>
+                        <mu>0.7</mu>
+                        <mu2>0.7</mu2>
+                        <fdir1>1 0 0</fdir1>
+                    </ode>
+                </friction>
+            </surface>
             <origin xyz="0 0 0" rpy="0 0 0"/>
             <geometry>
@@ -171,4 +221,13 @@
         </visual>
         <collision>
+            <surface>
+                <friction>
+                    <ode>
+                        <mu>0.7</mu>
+                        <mu2>0.7</mu2>
+                        <fdir1>1 0 0</fdir1>
+                    </ode>
+                </friction>
+            </surface>
             <origin xyz="0 0 0" rpy="0 0 0"/>
             <geometry>
@@ -190,4 +249,13 @@
         </visual>
         <collision>
+            <surface>
+                <friction>
+                    <ode>
+                        <mu>0.7</mu>
+                        <mu2>0.7</mu2>
+                        <fdir1>1 0 0</fdir1>
+                    </ode>
+                </friction>
+            </surface>
             <origin xyz="0 0 0" rpy="0 0 0"/>
             <geometry>
@@ -209,4 +277,13 @@
         </visual>
         <collision>
+            <surface>
+                <friction>
+                    <ode>
+                        <mu>0.7</mu>
+                        <mu2>0.7</mu2>
+                        <fdir1>1 0 0</fdir1>
+                    </ode>
+                </friction>
+            </surface>
             <origin xyz="0 0 0" rpy="0 0 0"/>
             <geometry>
@@ -229,4 +306,13 @@
         </visual>
         <collision>
+            <surface>
+                <friction>
+                    <ode>
+                        <mu>0.7</mu>
+                        <mu2>0.7</mu2>
+                        <fdir1>1 0 0</fdir1>
+                    </ode>
+                </friction>
+            </surface>
             <origin xyz="0 0 0" rpy="0 0 0"/>
             <geometry>
@@ -248,4 +334,13 @@
         </visual>
         <collision>
+            <surface>
+                <friction>
+                    <ode>
+                        <mu>0.7</mu>
+                        <mu2>0.7</mu2>
+                        <fdir1>1 0 0</fdir1>
+                    </ode>
+                </friction>
+            </surface>
             <origin xyz="0 0 0" rpy="0 0 0"/>
             <geometry>
@@ -267,4 +362,13 @@
         </visual>
         <collision>
+            <surface>
+                <friction>
+                    <ode>
+                        <mu>0.7</mu>
+                        <mu2>0.7</mu2>
+                        <fdir1>1 0 0</fdir1>
+                    </ode>
+                </friction>
+            </surface>
             <origin xyz="0 0 0" rpy="0 0 0"/>
             <geometry>
@@ -286,4 +390,13 @@
         </visual>
         <collision>
+            <surface>
+                <friction>
+                    <ode>
+                        <mu>0.7</mu>
+                        <mu2>0.7</mu2>
+                        <fdir1>1 0 0</fdir1>
+                    </ode>
+                </friction>
+            </surface>
             <origin xyz="0 0 0" rpy="0 0 0"/>
             <geometry>

File: description/lidar.xacro (robot description, xacro)
@@ -1,4 +1,13 @@
 <?xml version="1.0"?>
 <robot xmlns:xacro="http://www.ros.org/wiki/xacro" >
+    <xacro:macro name="inertial_sphere" params="mass radius *origin">
+        <inertial>
+            <xacro:insert_block name="origin"/>
+            <mass value="${mass}" />
+            <inertia ixx="${(2/5) * mass * (radius*radius)}" ixy="0.0" ixz="0.0"
+                    iyy="${(2/5) * mass * (radius*radius)}" iyz="0.0"
+                    izz="${(2/5) * mass * (radius*radius)}" />
+        </inertial>
+    </xacro:macro>
     <xacro:macro name="inertial_cylinder" params="mass length radius *origin">
         <inertial>
@@ -13,20 +22,19 @@
         <parent link="base_link"/>
         <child link="laser_frame"/>
-        <origin xyz="0.10 0 0.1" rpy="0 0 0"/>
+        <origin xyz="0.0 0 0.05" rpy="0 0 0"/>
     </joint>
     <link name="laser_frame">
         <visual>
             <geometry>
-                <cylinder radius="0.03" length="0.07"/>
-            </geometry>
-            <material name="black"/>
-        </visual>
-        <collision>
-            <geometry>
-                <origin xyz="0.03 0.03 0.03" rpy="0 0 0"/>
-                <cylinder radius="0.03" length="0.07"/>
-            </geometry>
-        </collision>
-        <xacro:inertial_cylinder mass="0.1" length="0.04" radius="0.05">
+                <cylinder radius="0.01" length="0.04"/>
+            </geometry>
+            <material name="black"/>
+        </visual>
+        <collision>
+            <geometry>
+                <cylinder radius="0.01" length="0.04"/>
+            </geometry>
+        </collision>
+        <xacro:inertial_cylinder mass="0.1" length="0.04" radius="0.1">
             <origin xyz="0 0 0" rpy="0 0 0"/>
         </xacro:inertial_cylinder>
@@ -48,5 +56,5 @@
                 <range>
                     <min>0.3</min>
-                    <max>12</max>
+                    <max>3</max>
                 </range>
             </ray>
@@ -60,3 +68,143 @@
         </sensor>
     </gazebo>
+<!--
+    <joint name="x_joint" type="fixed">
+        <parent link="base_link"/>
+        <child link="x_frame"/>
+        <origin xyz="0.10 0.05 0.07" rpy="0 0 0"/>
+    </joint>
+    <link name="x_frame">
+        <visual>
+            <origin xyz="0.0 0.05 0.06" rpy="0 0 0"/>
+            <geometry>
+                <cylinder radius="0.008" length="0.14"/>
+            </geometry>
+            <material name="black"/>
+        </visual>
+        <collision>
+            <origin xyz="0.0 0.05 0.06" rpy="0 0 0"/>
+            <geometry>
+                <cylinder radius="0.008" length="0.14"/>
+            </geometry>
+        </collision>
+        <xacro:inertial_cylinder mass="0.1" radius="0.008" length="0.14">
+            <origin xyz="0 0 0" rpy="0 0 0"/>
+        </xacro:inertial_cylinder>
+    </link>
+    <joint name="y_joint" type="fixed">
+        <parent link="base_link"/>
+        <child link="y_frame"/>
+        <origin xyz="0.10 -0.05 0.07" rpy="0 0 0"/>
+    </joint>
+    <link name="y_frame">
+        <visual>
+            <origin xyz="0.0 -0.05 0.06" rpy="0 0 0"/>
+            <geometry>
+                <cylinder radius="0.008" length="0.14"/>
+            </geometry>
+            <material name="black"/>
+        </visual>
+        <collision>
+            <origin xyz="0.0 -0.05 0.06" rpy="0 0 0"/>
+            <geometry>
+                <cylinder radius="0.008" length="0.14"/>
+            </geometry>
+        </collision>
+        <xacro:inertial_cylinder mass="0.1" radius="0.008" length="0.14">
+            <origin xyz="0 0 0" rpy="0 0 0"/>
+        </xacro:inertial_cylinder>
+    </link>
+    <joint name="z_joint" type="fixed">
+        <parent link="base_link"/>
+        <child link="z_frame"/>
+        <origin xyz="-0.06 -0.05 0.07" rpy="0 0 0"/>
+    </joint>
+    <link name="z_frame">
+        <visual>
+            <origin xyz="-0.060 -0.05 0.06" rpy="0 0 0"/>
+            <geometry>
+                <cylinder radius="0.008" length="0.14"/>
+            </geometry>
+            <material name="black"/>
+        </visual>
+        <collision>
+            <origin xyz="-0.060 -0.05 0.06" rpy="0 0 0"/>
+            <geometry>
+                <cylinder radius="0.08" length="0.14"/>
+            </geometry>
+        </collision>
+        <xacro:inertial_cylinder mass="0.1" radius="0.008" length="0.14">
+            <origin xyz="0 0 0" rpy="0 0 0"/>
+        </xacro:inertial_cylinder>
+    </link>
+    <joint name="w_joint" type="fixed">
+        <parent link="base_link"/>
+        <child link="w_frame"/>
+        <origin xyz="-0.060 0.05 0.07" rpy="0 0 0"/>
+    </joint>
+    <link name="w_frame">
+        <visual>
+            <origin xyz="-0.060 0.05 0.06" rpy="0 0 0"/>
+            <geometry>
+                <cylinder radius="0.008" length="0.14"/>
+            </geometry>
+            <material name="black"/>
+        </visual>
+        <collision>
+            <origin xyz="-0.060 0.05 0.06" rpy="0 0 0"/>
+            <geometry>
+                <cylinder radius="0.008" length="0.14"/>
+            </geometry>
+        </collision>
+        <xacro:inertial_cylinder mass="0.1" radius="0.008" length="0.14">
+            <origin xyz="0 0 0" rpy="0 0 0"/>
+        </xacro:inertial_cylinder>
+    </link>  -->
+<!--
+    <joint name="a_joint" type="fixed">
+        <parent link="base_link"/>
+        <child link="a_frame"/>
+        <origin xyz="0 0.04 0.06" rpy="0 0 0"/>
+    </joint>
+    <link name="a_frame">
+        <visual>
+            <origin xyz="0 0.04 0.06" rpy="0 0 0"/>
+            <geometry>
+                <cylinder radius="0.009" length="0.15"/>
+            </geometry>
+            <material name="black"/>
+        </visual>
+        <collision>
+            <origin xyz="0 0.04 0.06" rpy="0 0 0"/>
+            <geometry>
+                <cylinder radius="0.009" length="0.15"/>
+            </geometry>
+        </collision>
+        <xacro:inertial_cylinder mass="0.3" radius="0.005" length="0.1">
+            <origin xyz="0 0 0" rpy="0 0 0"/>
+        </xacro:inertial_cylinder>
+    </link>
+    <joint name="b_joint" type="fixed">
+        <parent link="base_link"/>
+        <child link="b_frame"/>
+        <origin xyz="0 -0.04 0.06" rpy="0 0 0"/>
+    </joint>
+    <link name="b_frame">
+        <visual>
+            <origin xyz="0 -0.04 0.06" rpy="0 0 0"/>
+            <geometry>
+                <cylinder radius="0.009" length="0.15"/>
+            </geometry>
+            <material name="black"/>
+        </visual>
+        <collision>
+            <origin xyz="0 -0.04 0.05" rpy="0 0 0"/>
+            <geometry>
+                <cylinder radius="0.009" length="0.15"/>
+            </geometry>
+        </collision>
+        <xacro:inertial_cylinder mass="0.3" radius="0.005" length="0.1">
+            <origin xyz="0 0 0" rpy="0 0 0"/>
+        </xacro:inertial_cylinder>
+    </link> -->
 </robot>
